File: cypress_logic_analyzer.sch (KiCad schematic (older format))
At the start: 12 parts, among them P1 CONN_02X10, P2 CONN_02X10, P3 CONN_01X09, U1 74LCX245

Commit message: Rev1.1, fixed routing, added decoupling cap
Parts:
- added C1: .1uF, Capacitors_SMD:C_0805_HandSoldering, symbol C
Changed lines of the file:
@@
 Text Label 4550 2250 1    60   ~ 0
 PB7
+$Comp
+L C C1
+U 1 1 5572932A
+P 2200 2650
+F 0 "C1" H 2225 2750 50  0000 L CNN
+F 1 ".1uF" H 2225 2550 50  0000 L CNN
+F 2 "Capacitors_SMD:C_0805_HandSoldering" H 2238 2500 30  0001 C CNN
+F 3 "" H 2200 2650 60  0000 C CNN
+	1    2200 2650
+	1    0    0    -1
+$EndComp
+$Comp
+L GND #PWR06
+U 1 1 55729375
+P 2200 2800
+F 0 "#PWR06" H 2200 2550 50  0001 C CNN
+F 1 "GND" H 2200 2650 50  0000 C CNN
+F 2 "" H 2200 2800 60  0000 C CNN
+F 3 "" H 2200 2800 60  0000 C CNN
+	1    2200 2800
+	1    0    0    -1
+$EndComp
+Connection ~ 2200 2500
+Connection ~ 2200 2800
 $EndSCHEMATC
